Commit message: update the marker task world

File: ur3_gazebo/urdf/ur_rstest.xacro (robot description, xacro)
@@ -59,5 +59,5 @@
   <xacro:include filename="$(find ur3_description)/urdf/camera/realsense_rs435_wrist.urdf.xacro" />
   <sensor_d435 parent="wrist_3_link">
-    <origin xyz="0 0.035 -0.03" rpy="0 -${pi/2} -${pi/2}" />
+    <origin xyz="0 0.040 -0.020" rpy="0 -${pi*120/180} -${pi/2}" />
   </sensor_d435>
   <!--

Commit message: robot follow marker

File: ur3_gazebo/urdf/ur_rstest.xacro (robot description, xacro)
@@ -60,4 +60,5 @@
   <sensor_d435 parent="wrist_3_link">
     <origin xyz="0 0.040 -0.020" rpy="0 -${pi*120/180} -${pi/2}" />
+    <!-- <origin xyz="0 0 0" rpy="0 0 0" /> -->
   </sensor_d435>
   <!--
